File: kicad/esc.kicad_sch (KiCad schematic)
At the start: 2 parts, among them J4 Conn_01x03, J5 Conn_01x02

Commit message: PCB v2
Parts:
- removed J4: Conn_01x03, Connector_JST:JST_XH_B3B-XH-A_1x03_P2.50mm_Vertical, symbol Connector_Generic:Conn_01x03
- removed J5: Conn_01x02, Connector_AMASS:AMASS_XT60PW-F_1x02_P7.20mm_Horizontal, symbol Connector_Generic:Conn_01x02
- added H4, H7: MountingHole_Pad, holes:SMTSOM340, symbol Mechanical:MountingHole_Pad
Connections:
- net GND: now also H7.1
- net VCC: now also H4.1
