File: kicad/inertia.kicad_sch (KiCad schematic)
At the start: 29 parts, among them J10 Conn_01x02, J2 USB_C_Receptacle_USB2.0_16P, J3 Conn_01x02, SW1 SW_Push, SW2 SW_Push, U1 TJA1042T-3, U2 ESP32-S3-WROOM-1, U3 LSM6DSOTR

Commit message: PCB v2
Parts:
- removed J10: Conn_01x02, Connector_JST:JST_XH_B2B-XH-A_1x02_P2.50mm_Vertical, symbol Connector_Generic:Conn_01x02
- removed JCAN1, JCAN2: Conn_01x02, Connector_JST:JST_ZH_B2B-ZR_1x02_P1.50mm_Vertical, symbol Connector_Generic:Conn_01x02
- removed SW1, SW2: SW_Push, Button_Switch_THT:SW_PUSH_6mm_H5mm, symbol Switch:SW_Push
- removed TP2, TP3, TP4, TP5: TestPoint, TestPoint:TestPoint_Pad_D1.0mm, symbol Connector:TestPoint
- removed U2: ESP32-S3-WROOM-1, RF_Module:ESP32-S3-WROOM-1U, symbol RF_Module:ESP32-S3-WROOM-1
- added C2: 100nF 6.3V, Capacitor_SMD:C_0805_2012Metric, symbol Device:C
- added D7: ESD5Z3.3T1G, Diode_SMD:D_SOD-523, symbol Device:D
- added J11: Conn_01x02, Connector_JST:JST_XH_B2B-XH-A_1x02_P2.50mm_Vertical, symbol Connector_Generic:Conn_01x02
- added J4: Conn_01x04, Connector_JST:JST_XH_B4B-XH-AM_1x04_P2.50mm_Vertical, symbol Connector_Generic:Conn_01x04
- added J5: tf01A, TF01A:TF-01A, symbol Connector:Micro_SD_Card_Det1
- added JCAN1, JCAN2: S2B-ZR-SM, jst:S2B-ZR-SMxA, symbol Connector_Generic_MountingPin:Conn_01x02_MountingPin
- added JP1: SolderJumper_3_Open, Jumper:SolderJumper-3_P1.3mm_Open_RoundedPad1.0x1.5mm, symbol Jumper:SolderJumper_3_Open
- added SW1, SW2: TS-1088-AR02016, Button_Switch_SMD:SW_SPST_TS-1088-xR020, symbol Switch:SW_SPST
- added U1: ESP32-C5-WROOM-1, PCM_Espressif:ESP32-C5-WROOM-1, symbol Espressif:ESP32-C5-WROOM-1
- added U4: OTOS Robotronik, otos:OTOS_robotronik, symbol otos:otos_robotronik
- C1: value C -> 10uF 6.3V
- J2: value USB_C_Receptacle_USB2.0_16P -> 7010A
- TP1: footprint TestPoint:TestPoint_Pad_D1.0mm -> Connector_PinHeader_2.54mm:PinHeader_1x01_P2.54mm_Vertical
- U3: footprint LGA-14L_2P5X3X0P86_STM -> LSM6DSO:LGA-14L_2P5X3X0P86_STM
- renumbered U1 to U2
Connections:
- net +5V: now also JP1.3 (B)
- net BOOT: now also SW2.2 (B), U1.15 (GPIO28)
- net CAN+: now also JCAN1.1 (Pin_1), JCAN2.1 (Pin_1)
- net CAN-: now also JCAN1.2 (Pin_2), JCAN2.2 (Pin_2)
- net CANRX: now also U1.18 (GPIO27)
- net CANSTB: now also U1.19 (GPIO15)
- net CANTX: now also U1.21 (GPIO23)
- net D+: now also U1.14 (GPIO14/USB_D+)
- net D-: now also U1.13 (GPIO13/USB_D-)
- net EN: now also C2.1, SW1.2 (B), U1.3 (EN/CHIP_PU)
- net GND: now also J2.SH (SHIELD), C2.2, D7.2 (A), J4.4 (Pin_4), J5.10 (SHIELD), J5.6 (VSS), JCAN1.MP (MountPin), JCAN2.MP (MountPin), SW1.1 (A), SW2.1 (A), U1.1 (GND), U1.28 (GND), U1.29 (GND), U4.1 (GND); no longer J2.S1 (SHIELD)
- net GY_CS: now also U1.17 (GPIO4)
- net GY_INT: now also U1.8 (GPIO6)
- net MISO: now also J5.7 (DAT0), U1.23 (GPIO24)
- net MOSI: now also J5.3 (CMD), U1.27 (GPIO26)
- net RGBLED: now also U1.4 (GPIO2)
- net SCLK: now also J5.5 (CLK), U1.26 (GPIO25)
- net at D2.2 (DOUT): now also TP1.1
- net +3.3V renamed +3V3
- net +3V3: now also D7.1 (K), J5.4 (VDD), JP1.1 (A), U1.2 (3V3), U4.2 (+3V3)
- new net: J4.1 (Pin_1), JP1.2 (C)
- new net GPIO0: J11.2 (Pin_2), U1.6 (GPIO0)
- new net GPIO1: J11.1 (Pin_1), U1.7 (GPIO1)
- new net OTOS_RX: U1.12 (GPIO10), U4.6 (RX)
- new net OTOS_TX: U1.11 (GPIO9), U4.5 (TX)
- new net SCL: U1.10 (GPIO8), U4.4 (SCL)
- new net SDA: U1.9 (GPIO7), U4.3 (SDA)
- new net SD_CS: J5.2 (DAT3/CD), U1.5 (GPIO3)
- new net SD_DET: J5.9 (DET), U1.16 (GPIO5)
- new net U0RXD: J4.2 (Pin_2), U1.24 (U0RXD/GPIO12)
- new net U0TXD: J4.3 (Pin_3), U1.25 (U0TXD/GPIO11)
- no-connect marks 16 -> 9
Other:
- sheet esc1 ports: added none; removed ESC, RX, TX
- sheet esc2 ports: added none; removed ESC, RX, TX
- sheet esc3 ports: added none; removed ESC, RX, TX
- note added: "!padne CURRENT i=50A f=H4.1 t=H7.1 !padne CURRENT i=50A f=H5.1 t=H8.1 !padne CURRENT i=50A f=H6.1 t=H9.1 !padne VOLTAGE v=12V p=J3.2 n=J3.1"
- note added: "JTAG"
- moved on the sheet: R1
